Commit message: launch in aworld

File: auto_bot/description/robot.urdf.xacro (robot description, xacro)
@@ -1,5 +1,6 @@
 <?xml version="1.0"?>
 <robot xmlns:xacro="http://www.ros.org/wiki/xacro" name="robot">
-<!-- <link name="base_link"></link> -->
-    <xacro:include filename="robot_core.xacro"/>
+    <!-- <link name="base_link"></link> -->
+    <xacro:include filename="robot_core.xacro" />
+    <xacro:include filename="gazebo_control.xacro" />
 </robot>

File: auto_bot/description/robot_core.xacro (robot description, xacro)
@@ -41,4 +41,7 @@
         <origin xyz="-0.1 0 0" rpy="0 0 0"/>
     </joint>
+    <gazebo reference="chassis_link">
+        <material>Gazebo/White</material>
+    </gazebo>
     <!-- Left Wheel Link -->
     <link name="left_wheel_link">
@@ -66,4 +69,7 @@
         <axis xyz="0 0 1"/>
     </joint>
+    <gazebo reference="left_wheel_link">
+        <material>Gazebo/Blue</material>
+    </gazebo>
     <!-- Right Wheel Link -->
     <link name="right_wheel_link">
@@ -91,4 +97,7 @@
         <axis xyz="0 0 -1"/>
     </joint>
+    <gazebo reference="right_wheel_link">
+        <material>Gazebo/Blue</material>
+    </gazebo>
     <!-- In this configuration y-axis of right will be up and keft will be down we want the z-axis of both to point outward -->
     <!-- Caster Wheel Link -->
@@ -116,3 +125,8 @@
         <origin xyz="0.24 0 0" rpy="0 0 0"/>
     </joint>
+    <gazebo reference="caster_link">
+        <material>Gazebo/Black</material>
+        <mu1 value="0.001"/>
+        <mu2 value="0.001"/>
+    </gazebo>
 </robot>
