Commit message: hardware interface & SLAM

File: auto_bot/description/robot_core.xacro (robot description, xacro)
@@ -17,4 +17,11 @@
     <link name="base_link">
     </link>
+    <!-- Base footprint link -->
+    <link name="base_footprint"></link>
+    <joint name="base_footprint_joint" type="fixed">
+        <parent link="base_link"/>
+        <child link="base_footprint"/>
+        <origin xyz="0 0 0" rpy="0 0 0"/>
+    </joint>
     <!-- Chassis Link -->
     <link name="chassis_link">
